File: SIM7020E/SIM7020E.sch (KiCad schematic (older format))
At the start: 45 parts, among them J1 Conn_01x03, J2 SIM_Card, J3 Conn_01x02, Q1 Q_NPN_BCE, Q2 Q_NPN_BCE, Q3 Q_NPN_BCE, Q4 Q_NPN_BCE, Q5 Q_NPN_BCE, Q6 Q_NPN_BCE, SW1 SW_Push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

Commit message: pcb update
Parts:
- AE1: footprint (none) -> Connector_Coaxial:U.FL_Molex_MCRF_73412-0110_Vertical
- C1, C10, C11, C2, C3, C4, C8, C9: footprint (none) -> Capacitor_SMD:C_0603_1608Metric_Pad1.05x0.95mm_HandSolder
- C5, C6, C7: footprint (none) -> Capacitor_Tantalum_SMD:CP_EIA-3528-21_Kemet-B_Pad1.50x2.35mm_HandSolder
- D1, D3: footprint (none) -> LED_SMD:LED_0603_1608Metric_Pad1.05x0.95mm_HandSolder
- D2: footprint (none) -> Diode_SMD:D_SOD-323_HandSoldering
- J1: footprint (none) -> Connector_PinSocket_2.54mm:PinSocket_1x03_P2.54mm_Vertical
- J2: footprint (none) -> Connector_Card:GCT_SIM8051-6-0-14-00-X-REVD
- J3: footprint (none) -> Connector_PinHeader_2.54mm:PinHeader_1x02_P2.54mm_Vertical
- Q1, Q2, Q3, Q4, Q5, Q6: footprint (none) -> Package_TO_SOT_SMD:SOT-23
- R1, R10, R12, R13, R4, R5, R7, R9: footprint (none) -> Resistor_SMD:R_0805_2012Metric_Pad1.15x1.40mm_HandSolder
- R11, R14, R15, R16, R17, R2, R3, R6, R8: footprint (none) -> Resistor_SMD:R_0603_1608Metric_Pad1.05x0.95mm_HandSolder
- SW1, SW2: footprint (none) -> Button_Switch_SMD:SW_SPST_CK_RS282G05A3
- U1: footprint (none) -> SIM:SIM7020E
